Commit message: Update macro.m1013.white.xacro

File: dsr_description2/xacro/macro.m1013.white.xacro (robot description, xacro)
@@ -185,5 +185,5 @@
 			<parent link="link5" />
 			<child link="link6" />
-			<origin rpy="1.571 0 0" xyz="0 -0.124 0" />
+			<origin rpy="1.571 0 0" xyz="0 -0.121 0" />
 			<axis xyz="0 0 1" />
 			<limit effort="50" lower="-6.2832" upper="6.2832" velocity="3.927"/>
